File: PCE_Colorlight_Carrier/core.kicad_sch (KiCad schematic)
At the start: 19 parts, among them J5 POGO, T2 HX5008, U17 Colorlight i5 v7.0

Commit message: Add files via upload
Parts:
- T2: footprint HX5008:HX5008NL -> Library:SOP-24_L13.2-W15.1-P0.99-LS18.7-BL
