File: PCE_Colorlight_Carrier/front_io.kicad_sch (KiCad schematic)
At the start: 87 parts, among them J3 HuCard_38pin, SW2 HX 5.2X5.2X2.0H SWITCH TACTIL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, SW3 HX 5.2X5.2X2.0H SWITCH TACTIL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, SW4 HX 5.2X5.2X2.0H SWITCH TACTIL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, U1 TXB0108PWR, U12 74LVC8T245PW_C52140502, U13 74LVC8T245PW_C52140502, U15 DIN PLAYER 1, U16 TXB0108PWR, U18 DIN PLAYER 2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

Commit message: Add files via upload
Parts:
- added C78, C79: 100 nF, Capacitor_SMD:C_0402_1005Metric, symbol Device:C_Small
- U12, U13, U2, U3: footprint Library:74LVC245APW -> Library:TSSOP-24_L7.8-W4.4-P0.65-LS6.4-BL_1
Connections:
- net +3.3V_SYS: now also C79.1
- net +5V_SYS: now also C78.1
- net GND: now also C78.2, C79.2
