File: PCE_Colorlight_Carrier/power.kicad_sch (KiCad schematic)
At the start: 19 parts, among them SW1 TK-6580A-1, U14 SY8205FCC

Commit message: Add files via upload
Connections:
- net GND: now also USBC1.1 (EH), USBC1.2 (EH), USBC1.3 (EH), USBC1.4 (EH)
- net at SW1.1: no longer F1.1
- net at SW1.3: now also F1.1
