File: PCE_Colorlight_Carrier/usb_JTAG-UART.kicad_sch (KiCad schematic)
At the start: 32 parts, among them J6 USB_JTAG-UART, J7 POGO, U21 NUP2202, U24 FT2232HL, U6 93CxxC, Y2 12MHZ

Commit message: Add files via upload
Parts:
- removed J6: USB_JTAG-UART, USB-C-COM-15111:USB-C-COM-15111, symbol usb_c16pin:USB_C16PIN
- added USBC2: TYPE-C-31-M-12, Library:USB-C_SMD-TYPE-C-31-M-12_1, symbol perso:TYPE-C-31-M-12
- FB1, FB2: footprint Inductor_SMD:L_0805_2012Metric_Pad1.15x1.40mm_HandSolder -> Fuse:Fuse_0805_2012Metric_Pad1.15x1.40mm_HandSolder
Connections:
- net +5V JTAG-UART: now also USBC2.A4B9 (VBUS), USBC2.B4A9 (VBUS)
- net GND: now also USBC2.1 (EH), USBC2.2 (EH), USBC2.3 (EH), USBC2.4 (EH), USBC2.A1B12 (GND), USBC2.B1A12 (GND)
- net at R34.1, U21.6: now also USBC2.A6 (DP1), USBC2.B6 (DP2)
- net at R38.1, U21.1: now also USBC2.A7 (DN1), USBC2.B7 (DN2)
- no-connect marks 28 -> 30
