File: PCE_Colorlight_Carrier/usb_host.kicad_sch (KiCad schematic)
At the start: 46 parts, among them J4 SWD, Q1 Q12MHz/20pF/10ppm/4P/3.2x2.5mm, SW6 SW_Push, U19 CH217K(SOT23-6L), U20 CH334S(SSOP-28), U23 USBLC6-2SC6, U25 USBLC6-2SC6, U26 USBLC6-2SC6, U27 USBLC6-2SC6, U5 RP2040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

Commit message: Add files via upload
Parts:
- removed SW6: SW_Push, Connector_PinSocket_2.54mm:PinSocket_1x02_P2.54mm_Vertical, symbol Switch:SW_Push
- removed USB_HOST2: USBB1-FRWH-4A(USB-Ax2), OLIMEX_Connectors-FP:USB_TWO_LEVEL, symbol OLIMEX_Connectors:USB_HOST-TWO_LEVEL
- added SW5: HX 5.2X5.2X2.0H SWITCH TACTILE SPST-NO 0.05A 12V, Library:SW-SMD, symbol perso:HX5.2X5.2X2.0HSWITCHTACTILESPST-NO0.05A12V
- added USB_HOST2: USBB1-FRWH-4A(USB-Ax2), Library:USB-A-TH_USB-269-BRW, symbol perso:USB-269-BRW
- C14, C21, C29, C30, C31: footprint OLIMEX_RLC-FP:C_0805_5MIL_DWS -> PCM_4ms_Capacitor:C_0603
- C15, C16: footprint OLIMEX_RLC-FP:C_0603_5MIL_DWS -> PCM_4ms_Capacitor:C_0603
- C17, C18, C19: footprint OLIMEX_RLC-FP:C_0402_5MIL_DWS -> PCM_4ms_Capacitor:C_0603
- R32: footprint OLIMEX_RLC-FP:R_0402_5MIL_DWS -> PCM_4ms_Resistor:R_0603
- U19: footprint OLIMEX_IC-FP:SOT23-6 -> Library:SOT-23-6_L2.9-W1.6-P0.95-LS2.8-BL
- U20: footprint OLIMEX_IC-FP:SSOP28 -> Library:SSOP-28_L10.2-W5.3-P0.65-LS7.8-BL
- USB_HOST1: footprint OLIMEX_Connectors-FP:USB_TWO_LEVEL -> Library:USB-A-TH_USB-269-BRW; symbol OLIMEX_Connectors:USB_HOST-TWO_LEVEL -> perso:USB-269-BRW; LCSC Part (none) -> C720548; MPN (none) -> USB-269-BRW; Manufacturer (none) -> XUNPU(讯普)
Connections:
- net +5V: now also USB_HOST1.1 (VBUS), USB_HOST1.5 (VBUS), USB_HOST2.1 (VBUS), USB_HOST2.6 (D-); no longer USB_HOST1.1.1, USB_HOST1.2.1
- net GND: now also USB_HOST1.10 (GND), USB_HOST1.11 (GND), USB_HOST1.12 (GND), USB_HOST1.4 (GND), USB_HOST1.8 (GND), USB_HOST1.9 (GND), SW5.1, USB_HOST2.10 (GND), USB_HOST2.11 (GND), USB_HOST2.12 (GND), USB_HOST2.4 (GND), USB_HOST2.9 (GND); no longer USB_HOST1.0, USB_HOST1.1.4, USB_HOST1.2.4
- net USB_D+: now also R39.2; no longer R39.1, U5.47 (USB_DP)
- net USB_D-: now also R40.2; no longer R40.1, U5.46 (USB_DM)
- net USB_D1+: now also USB_HOST1.3 (D+); no longer USB_HOST1.1.3
- net USB_D1-: now also USB_HOST1.2 (D-); no longer USB_HOST1.1.2
- net USB_D2+: now also USB_HOST1.7 (D+); no longer USB_HOST1.2.3
- net USB_D2-: now also USB_HOST1.6 (D-); no longer USB_HOST1.2.2
- net USB_D3+: now also USB_HOST2.3 (D+)
- net USB_D3-: now also USB_HOST2.2 (D-)
- net USB_D4+: now also USB_HOST2.8 (GND)
- net USB_D4-: now also USB_HOST2.7 (D+)
- net ~{USB_BOOT}: now also SW5.4
- new net: R40.1, U5.46 (USB_DM)
- new net: R39.1, U5.47 (USB_DP)
